Commit message: feat: lidar 위치 조정 & RGBD camera 추가

File: go2_description/xacro/robot_VLP.xacro (robot description, xacro)
@@ -112,3 +112,4 @@
     <xacro:include filename="$(find go2_description)/xacro/velodyne.xacro"/>
     <!-- <xacro:include filename="$(find go2_description)/xacro/laser.xacro"/> -->
+    <xacro:include filename="$(find go2_description)/xacro/realsense_rgbd.xacro"/>
 </robot>

File: go2_description/xacro/velodyne.xacro (robot description, xacro)
@@ -2,5 +2,5 @@
 <robot xmlns:xacro="http://www.ros.org/wiki/xacro">
     <joint name="velodyne_base_mount_joint" type="fixed">
-        <origin rpy="0 0 0" xyz="0.2 0 0.08"/>
+        <origin rpy="0 0 0" xyz="-0.05 0 0.08"/>
         <parent link="base_link"/>
         <child link="velodyne_base_link"/>
